File: AmpliGSR/AmpliGSR.kicad_pcb (KiCad board)
At the start: 2 copper layers, 40.6 x 33 mm, 16 parts, among them P1 CONN_01X01, P2 CONN_01X01, P3 CONN_01X03, U1 LM324N

Commit message: update ampli schematic & pcb
Parts:
- added C3: 10u, Capacitors_ThroughHole:C_Radial_D5_L11_P2, F.Cu at (148.6, 116.2)
- R5: value 10k -> 150k
- moved R8 13.9 mm to (132.7, 125.7), turned to 180 degrees
- moved P2 5.39 mm to (151.1, 120.7)
- moved P1 4.26 mm to (151.1, 126.4)
Routing:
- net Net-(R8-Pad1): track 34.4 -> 22.0 mm
- net GND: track 72.4 -> 82.9 mm
- net Net-(C2-Pad1): track 64.9 -> 71.6 mm
- net Net-(C1-Pad2): track 10.2 -> 15.1 mm
- net Net-(R8-Pad2): track 5.08 -> 9.02 mm
