File: AmpliGSR/AmpliGSR.sch (KiCad schematic (older format))
At the start: 16 parts, among them P1 CONN_01X01, P2 CONN_01X01, P3 CONN_01X03, U1 LM324N

Commit message: update ampli schematic & pcb
Parts:
- added C3: 10u, Capacitors_ThroughHole:C_Radial_D5_L11_P2, symbol CP2
- R3, R4: value 2.2k -> 10k
- R5: value 47k -> 150k
Connections:
- net GND: now also C3.2
- net at C1.2, P3.1 (P1), R10.1: now also C3.1
Other:
- moved on the sheet: P3
Changed lines of the file:
@@
 EESchema Schematic File Version 2
-LIBS:power
 LIBS:device
-LIBS:transistors
-LIBS:conn
-LIBS:linear
-LIBS:regul
-LIBS:74xx
-LIBS:cmos4000
-LIBS:adc-dac
-LIBS:memory
-LIBS:xilinx
-LIBS:special
-LIBS:microcontrollers
-LIBS:dsp
-LIBS:microchip
-LIBS:analog_switches
-LIBS:motorola
-LIBS:texas
-LIBS:intel
-LIBS:audio
-LIBS:interface
-LIBS:digital-audio
-LIBS:philips
-LIBS:display
-LIBS:cypress
-LIBS:siliconi
-LIBS:opto
-LIBS:atmel
-LIBS:contrib
-LIBS:valves
 LIBS:AmpliGSR-cache
 EELAYER 25 0
@@
 P 2950 1650
 F 0 "R3" V 3030 1650 40  0000 C CNN
-F 1 "2.2k" V 2957 1651 40  0000 C CNN
+F 1 "10k" V 2957 1651 40  0000 C CNN
 F 2 "Resistors_ThroughHole:Resistor_Horizontal_RM7mm" V 2880 1650 30  0001 C CNN
 F 3 "" H 2950 1650 30  0000 C CNN
@@
 P 2950 2200
 F 0 "R4" V 3030 2200 40  0000 C CNN
-F 1 "2.2k" V 2957 2201 40  0000 C CNN
+F 1 "10k" V 2957 2201 40  0000 C CNN
 F 2 "Resistors_ThroughHole:Resistor_Horizontal_RM7mm" V 2880 2200 30  0001 C CNN
 F 3 "" H 2950 2200 30  0000 C CNN
@@
 P 2950 1100
 F 0 "R5" V 3030 1100 40  0000 C CNN
-F 1 "47k" V 2957 1101 40  0000 C CNN
+F 1 "150k" V 2957 1101 40  0000 C CNN
 F 2 "Resistors_ThroughHole:Resistor_Horizontal_RM7mm" V 2880 1100 30  0001 C CNN
 F 3 "" H 2950 1100 30  0000 C CNN
@@
 $EndComp
 Wire Wire Line
-	6900 2000 7350 2000
+	6900 2000 7650 2000
 Wire Wire Line
 	6950 2050 6950 2000
@@
 L CONN_01X03 P3
 U 1 1 574C43EF
-P 7550 2100
-F 0 "P3" H 7550 2300 50  0000 C CNN
-F 1 "CONN_01X03" V 7650 2100 50  0000 C CNN
-F 2 "Connectors_Molex:Molex_KK_6410-03" H 7550 2100 60  0001 C CNN
-F 3 "" H 7550 2100 60  0000 C CNN
-	1    7550 2100
+P 7850 2100
+F 0 "P3" H 7850 2300 50  0000 C CNN
+F 1 "CONN_01X03" V 7950 2100 50  0000 C CNN
+F 2 "Connectors_Molex:Molex_KK_6410-03" H 7850 2100 60  0001 C CNN
+F 3 "" H 7850 2100 60  0000 C CNN
+	1    7850 2100
 	1    0    0    -1
 $EndComp
@@
 L GND #PWR09
 U 1 1 574C4461
-P 7350 2250
-F 0 "#PWR09" H 7350 2250 30  0001 C CNN
-F 1 "GND" H 7350 2180 30  0001 C CNN
-F 2 "" H 7350 2250 60  0000 C CNN
-F 3 "" H 7350 2250 60  0000 C CNN
-	1    7350 2250
+P 7650 2250
+F 0 "#PWR09" H 7650 2250 30  0001 C CNN
+F 1 "GND" H 7650 2180 30  0001 C CNN
+F 2 "" H 7650 2250 60  0000 C CNN
+F 3 "" H 7650 2250 60  0000 C CNN
+	1    7650 2250
 	1    0    0    -1
 $EndComp
@@
 L +5V #PWR010
 U 1 1 574C4517
-P 7300 2100
-F 0 "#PWR010" H 7300 2190 20  0001 C CNN
-F 1 "+5V" H 7300 2190 30  0000 C CNN
-F 2 "" H 7300 2100 60  0000 C CNN
-F 3 "" H 7300 2100 60  0000 C CNN
-	1    7300 2100
+P 7600 2100
+F 0 "#PWR010" H 7600 2190 20  0001 C CNN
+F 1 "+5V" H 7600 2190 30  0000 C CNN
+F 2 "" H 7600 2100 60  0000 C CNN
+F 3 "" H 7600 2100 60  0000 C CNN
+	1    7600 2100
 	0    -1   -1   0
 $EndComp
 Wire Wire Line
-	7300 2100 7350 2100
-Wire Wire Line
-	7350 2200 7350 2250
+	7600 2100 7650 2100
+Wire Wire Line
+	7650 2200 7650 2250
 Text Notes 1850 3600 0    60   ~ 0
 VG = VS * ([Rx /{R4 + Rx}] – [R5/{R3 + R5}])\n       = 0.5 * ( Rx/(2k + Rx) - 0.96)
+$Comp
+L CP2 C3
+U 1 1 57CEF5FA
+P 7150 2200
+F 0 "C3" H 7150 2300 40  0000 L CNN
+F 1 "10u" H 7156 2115 40  0000 L CNN
+F 2 "Capacitors_ThroughHole:C_Radial_D5_L11_P2" H 7188 2050 30  0001 C CNN
+F 3 "" H 7150 2200 60  0000 C CNN
+	1    7150 2200
+	1    0    0    -1
+$EndComp
+$Comp
+L GND #PWR011
+U 1 1 57CEF81F
+P 7150 2450
+F 0 "#PWR011" H 7150 2450 30  0001 C CNN
+F 1 "GND" H 7150 2380 30  0001 C CNN
+F 2 "" H 7150 2450 60  0000 C CNN
+F 3 "" H 7150 2450 60  0000 C CNN
+	1    7150 2450
+	1    0    0    -1
+$EndComp
+Wire Wire Line
+	7150 2450 7150 2400
+Connection ~ 7150 2000
 $EndSCHEMATC
